File: kicad/iris.kicad_pcb (KiCad board)
At the start: 2 copper layers, 42 x 120 mm, 23 parts, among them U1 XIAO-RP2040-SMD

Commit message: feat: add silkscreen art to pcb
Parts:
- added G***: LOGO, LOGO, F.Cu at (45.8, 101.8)
- added G***: LOGO, LOGO, F.Cu at (54.9, 101.5)
- added G***: LOGO, LOGO, F.Cu at (57.1, 123.8)
- added G***: LOGO, LOGO, F.Cu at (57.1, 116.7)
- added G***: LOGO, LOGO, F.Cu at (55.5, 137.4)
- added G***: LOGO, LOGO, F.Cu at (48.3, 138.0)
- added G***: LOGO, LOGO, F.Cu at (57.1, 102.4)
Routing:
- net COL1: track 87.0 -> 91.7 mm
- net ROW4: track 146.7 -> 148.2 mm
- net ROW3: track 113.5 -> 114.9 mm
- net ROW2: track 91.6 -> 92.7 mm
- net ROW1: track 69.7 -> 70.6 mm
- net ROW0: track 47.7 -> 48.5 mm

Commit message: feat: update case and pcb to near production ready
Parts:
- moved G*** 2.38 mm to (57.1, 104.8)
Connections:
- MX11 pad 1: unconnected-(MX11-Pad1) -> COL0
Routing:
- net COL0: track 89.4 -> 99.0 mm
- added copper zone on B.Cu, net GND
Changed lines of the file:
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@@
 			(layers "*.Cu" "B.Mask")
 			(remove_unused_layers no)
-			(net "unconnected-(MX11-Pad1)")
+			(net "COL0")
 			(pinfunction "1_1")
 			(pintype "passive")
@@
 	(footprint "LOGO"
 		(layer "F.Cu")
-		(at 57.15 102.39375)
+		(at 57.15 104.775)
 		(property "Reference" "G***"
 			(at 0 0 0)
@@
 	)
 	(segment
+		(start 52.86375 149.86)
+		(end 43.33875 149.86)
+		(width 0.2)
+		(layer "F.Cu")
+		(net "COL0")
+	)
+	(segment
 		(start 42.86175 149.383)
 		(end 43.33875 149.86)
@@
 		(net "ROW3")
 	)
+	(zone
+		(net "GND")
+		(layer "B.Cu")
+		(name "Ground")
+		(hatch edge 0.5)
+		(connect_pads
+			(clearance 0.5)
+		)
+		(min_thickness 0.25)
+		(fill yes
+			(thermal_gap 0.5)
+			(thermal_bridge_width 0.5)
+			(island_removal_mode 0)
+		)
+		(polygon
+			(pts
+				(xy 28.575 38.1) (xy 83.34375 38.1) (xy 83.34375 169.06875) (xy 28.575 169.06875)
+			)
+		)
+	)
 	(embedded_fonts no)

Commit message: feat: update case to v2 prototype
Parts:
- removed D11: SOD-123, Diode_SMD:D_SOD-123
Connections:
- MX11 pad 2: Net-(D11-A) -> Net-(D9-A)
Routing:
- net Net-(D9-A): track 11.0 -> 22.1 mm
- net ROW4: track 148.2 -> 137.8 mm
- net Net-(D11-A): track 8.32 -> 0.00 mm
