File: kicad/iris.kicad_sch (KiCad schematic)
At the start: 0 parts

Commit message: feat: finish pcb layout
Parts:
- added D1, D10, D11, D2, D3, D4, D5, D6, D7, D8, D9: SOD-123, Diode_SMD:D_SOD-123, symbol Device:D_Small
- added MX1, MX10, MX2, MX3, MX4, MX5, MX6, MX7, MX8, MX9: MX-NoLED, MX_Solderable:MX-Solderable-1U, symbol Switch:SW_Push_45deg
- added MX11: MX-NoLED, MX_Solderable:MX-Solderable-2U, symbol Switch:SW_Push_45deg
- added U1: XIAO-RP2040-SMD, xiao:XIAO-RP2040-DIP, symbol Seeed_Studio_XIAO_Series:XIAO-RP2040-SMD
Connections:
- new net: D4.2 (A), MX4.2
- new net: D10.2 (A), MX10.2
- new net: D6.2 (A), MX6.2
- new net: D2.2 (A), MX2.2
- new net: D7.2 (A), MX7.2
- new net: D8.2 (A), MX8.2
- new net: D11.2 (A), MX11.2
- new net: D5.2 (A), MX5.2
- new net: D3.2 (A), MX3.2
- new net: D9.2 (A), MX9.2
- new net: D1.2 (A), MX1.2
- new net COL0: MX1.1, MX3.1, MX5.1, MX7.1, MX9.1, U1.8 (GPIO1_D7_CSn_RX)
- new net COL1: MX10.1, MX2.1, MX4.1, MX6.1, MX8.1, U1.7 (GPIO0_D6_TX)
- new net GND: U1.13 (GND), U1.16 (GND), U1.20 (GND)
- new net ROW0: D1.1 (K), D2.1 (K), U1.6 (GPIO7_D5_SCL)
- new net ROW1: D3.1 (K), D4.1 (K), U1.5 (GPIO6_D4_SDA)
- new net ROW2: D5.1 (K), D6.1 (K), U1.4 (GPIO29_A3_D3)
- new net ROW3: D7.1 (K), D8.1 (K), U1.3 (GPIO28_A2_D2)
- new net ROW4: D10.1 (K), D11.1 (K), D9.1 (K), U1.2 (GPIO27_A1_D1)
- no-connect marks 0 -> 10

Commit message: feat: update case and pcb to near production ready
Connections:
- net COL0: now also MX11.1
Changed lines of the file:
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@@
+	)
+	(junction
+		(at 38.1 129.54)
+		(diameter 0)
+		(color 0 0 0 0)
 	)
 	(junction
@@
 	)
 	(junction
+		(at 54.61 52.07)
+		(diameter 0)
+		(color 0 0 0 0)
+	)
+	(junction
 		(at 38.1 109.22)
 		(diameter 0)
@@
 	)
 	(junction
-		(at 54.61 52.07)
-		(diameter 0)
-		(color 0 0 0 0)
-	)
-	(junction
 		(at 38.1 52.07)
 		(diameter 0)
@@
 	(wire
 		(pts
+			(xy 38.1 129.54) (xy 53.34 129.54)
+		)
+		(stroke
+			(width 0)
+			(type default)
+		)
+	)
+	(wire
+		(pts
+			(xy 53.34 129.54) (xy 53.34 132.08)
+		)
+		(stroke
+			(width 0)
+			(type default)
+		)
+	)
+	(wire
+		(pts
 			(xy 54.61 71.12) (xy 54.61 90.17)
 		)
@@
 	(wire
 		(pts
+			(xy 53.34 132.08) (xy 58.42 132.08)
+		)
+		(stroke
+			(width 0)
+			(type default)
+		)
+	)
+	(wire
+		(pts
 			(xy 43.18 63.5) (xy 59.69 63.5)
 		)
@@
 		)
 		(stroke
+			(width 0)
+			(type default)
+		)
+	)
+	(wire
+		(pts
+			(xy 58.42 129.54) (xy 67.31 129.54)
+		)
+		(stroke
+			(width 0)
+			(type default)
+		)
+	)
+	(wire
+		(pts
+			(xy 58.42 132.08) (xy 58.42 129.54)
+		)
+		(stroke

Commit message: feat: update case to v2 prototype
Parts:
- removed D11: SOD-123, Diode_SMD:D_SOD-123, symbol Device:D_Small
Connections:
- net at MX11.2: now also D9.2 (A), MX9.2
Other:
- moved on the sheet: MX11
Changed lines of the file:
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@@
+	)
+	(junction
+		(at 43.18 134.62)
+		(diameter 0)
+		(color 0 0 0 0)
 	)
 	(junction
@@
 	)
 	(junction
-		(at 38.1 129.54)
-		(diameter 0)
-		(color 0 0 0 0)
-	)
-	(junction
 		(at 59.69 63.5)
 		(diameter 0)
@@
 	)
 	(junction
-		(at 72.39 140.97)
+		(at 38.1 129.54)
 		(diameter 0)
 		(color 0 0 0 0)
@@
 	(wire
 		(pts
-			(xy 38.1 129.54) (xy 53.34 129.54)
-		)
-		(stroke
-			(width 0)
-			(type default)
-		)
-	)
-	(wire
-		(pts
-			(xy 53.34 129.54) (xy 53.34 132.08)
-		)
-		(stroke
-			(width 0)
-			(type default)
-		)
-	)
-	(wire
-		(pts
 			(xy 54.61 71.12) (xy 54.61 90.17)
 		)
@@
 	(wire
 		(pts
-			(xy 72.39 134.62) (xy 72.39 135.89)
+			(xy 33.02 134.62) (xy 43.18 134.62)
 		)
 		(stroke
@@
 	(wire
 		(pts
-			(xy 72.39 140.97) (xy 76.2 140.97)
-		)
-		(stroke
-			(width 0)
-			(type default)
-		)
-	)
-	(wire
-		(pts
-			(xy 53.34 132.08) (xy 58.42 132.08)
+			(xy 59.69 140.97) (xy 76.2 140.97)
 		)
 		(stroke
@@
 	(wire
 		(pts
-			(xy 58.42 129.54) (xy 67.31 129.54)
-		)
-		(stroke
-			(width 0)
-			(type default)
-		)
-	)
-	(wire
-		(pts
-			(xy 58.42 132.08) (xy 58.42 129.54)
+			(xy 27.94 129.54) (xy 38.1 129.54)
 		)
 		(stroke
@@
 		(pts
 			(xy 59.69 82.55) (xy 76.2 82.55)
-		)
-		(stroke
-			(width 0)
-			(type default)
-		)
-	)
-	(wire
-		(pts
-			(xy 59.69 140.97) (xy 72.39 140.97)
 		)
 		(stroke
@@
 	(symbol
 		(lib_id "Switch:SW_Push_45deg")
-		(at 69.85 132.08 0)
+		(at 30.48 132.08 0)
 		(unit 1)
 		(body_style 1)
@@
 		(fields_autoplaced yes)
 		(property "Reference" "MX11"
-			(at 69.85 124.46 0)
+			(at 30.48 124.46 0)
 			(show_name no)
 			(do_not_autoplace no)
@@
 		)
 		(property "Value" "MX-NoLED"
-			(at 69.85 127 0)
+			(at 30.48 127 0)
 			(show_name no)
 			(do_not_autoplace no)
@@
 		)
 		(property "Footprint" "MX_Solderable:MX-Solderable-2U"
-			(at 69.85 132.08 0)
+			(at 30.48 132.08 0)
 			(hide yes)
 			(show_name no)
@@
 		)
 		(property "Datasheet" ""
-			(at 69.85 132.08 0)
+			(at 30.48 132.08 0)
 			(hide yes)
 			(show_name no)
@@
 		)
 		(property "Description" "Push button switch, normally open, two pins, 45° tilted"
-			(at 69.85 132.08 0)
+			(at 30.48 132.08 0)
 			(hide yes)
 			(show_name no)
@@
 					(unit 1)
 				)
-			)
-		)
-	)
-	(symbol
-		(lib_id "Device:D_Small")
-		(at 72.39 138.43 90)
-		(unit 1)
-		(body_style 1)
-		(exclude_from_sim no)
-		(in_bom yes)
-		(on_board yes)
-		(in_pos_files yes)
-		(dnp no)
-		(fields_autoplaced yes)
-		(property "Reference" "D11"
-			(at 74.93 137.1599 90)
-			(show_name no)
-			(do_not_autoplace no)
-			(effects
-				(font
-					(size 1.27 1.27)
-				)
-				(justify right)
-			)
-		)
-		(property "Value" "SOD-123"
-			(at 74.93 139.6999 90)
-			(show_name no)
-			(do_not_autoplace no)
-			(effects
-				(font
-					(size 1.27 1.27)
-				)
-				(justify right)
-			)
-		)
-		(property "Footprint" "Diode_SMD:D_SOD-123"
-			(at 72.39 138.43 90)
-			(hide yes)
-			(show_name no)
-			(do_not_autoplace no)
-			(effects
-				(font
-					(size 1.27 1.27)
-				)
-			)
-		)
-		(property "Datasheet" ""
-			(at 72.39 138.43 90)
-			(hide yes)
-			(show_name no)
-			(do_not_autoplace no)
-			(effects
-				(font
-					(size 1.27 1.27)
-				)
-			)
-		)
-		(property "Description" "Diode, small symbol"
-			(at 72.39 138.43 0)
-			(hide yes)
-			(show_name no)
-			(do_not_autoplace no)
-			(effects
-				(font
-					(size 1.27 1.27)
-				)
-			)
-		)
-		(property "Sim.Device" "D"
-			(at 72.39 138.43 0)
-			(hide yes)
-			(show_name no)
-			(do_not_autoplace no)
-			(effects
-				(font
-					(size 1.27 1.27)
-				)
-			)
-		)
-		(property "Sim.Pins" "1=K 2=A"
-			(at 72.39 138.43 0)
-			(hide yes)
-			(show_name no)
-			(do_not_autoplace no)
-			(effects
-				(font
-					(size 1.27 1.27)
-				)
-			)
-		)
-		(pin "1"
-		)
-		(pin "2"
-		)
-		(instances
-			(project "iris"
-				(path "/202b2ab6-b70d-44cf-8ccd-cd620cd842be"
-					(reference "D11")
-					(unit 1)
-				)
